File: PCB/LO2SC.sch (KiCad schematic (older format))
At the start: 0 parts

Commit message: - ajout de schematiques
Parts:
- added P1, P2: CONN_01X05, Barrettes:Pin_Header_Straight_1x05, symbol CONN_01X05
Changed lines of the file:
@@
 LIBS:Resistances_SMD_0603
 LIBS:Condensateurs_SMD_0603
+LIBS:Microcontroleur_Atmel_SMD_TQFP
+LIBS:Barrettes_TH
 LIBS:LO2SC-cache
 EELAYER 25 0
@@
 $Descr A4 11693 8268
 encoding utf-8
-Sheet 1 2
+Sheet 1 5
 Title ""
 Date ""
@@
 S 1500 5300 2650 1350
 U 55FAC7CC
-F0 "Sheet55FAC7CB" 60
-F1 "Vitual Ground.sch" 60
+F0 "Out_Lineat+WideBand" 60
+F1 "Out_Lineat+WideBand.sch" 60
 $EndSheet
+$Sheet
+S 1500 4100 2650 1000
+U 55FBB281
+F0 "Sheet55FBB280" 60
+F1 "Arduino.sch" 60
+$EndSheet
+$Sheet
+S 1500 2900 2650 1000
+U 55FBEC71
+F0 "Sheet55FBEC70" 50
+F1 "Pump_RCAL.sch" 50
+$EndSheet
+$Sheet
+S 1500 1750 2650 1000
+U 55FBF4E6
+F0 "Sheet55FBF4E5" 50
+F1 "POUT_NARROW.sch" 50
+$EndSheet
+$Comp
+L CONN_01X05 P1
+U 1 1 55FBF5A3
+P 6150 2000
+F 0 "P1" H 6150 2300 50  0000 C CNN
+F 1 "CONN_01X05" V 6250 2000 50  0000 C CNN
+F 2 "Barrettes:Pin_Header_Straight_1x05" H 6150 2450 60  0001 C CNN
+F 3 "" H 6150 2300 60  0000 C CNN
+F 4 "455-1660-ND" H 6150 2550 50  0001 C CNN "Ref Digikey"
+	1    6150 2000
+	0    1    1    0
+$EndComp
+$Comp
+L CONN_01X05 P2
+U 1 1 55FBF5F9
+P 7000 1950
+F 0 "P2" H 7000 2250 50  0000 C CNN
+F 1 "CONN_01X05" V 7100 1950 50  0000 C CNN
+F 2 "Barrettes:Pin_Header_Straight_1x05" H 7000 2400 60  0001 C CNN
+F 3 "" H 7000 2250 60  0000 C CNN
+F 4 "455-1660-ND" H 7000 2500 50  0001 C CNN "Ref Digikey"
+	1    7000 1950
+	0    1    1    0
+$EndComp
 $EndSCHEMATC

Commit message: - routage
Parts:
- added U?: MIC5205-3.3YM5, SOT23-5, symbol MIC5205-3.3YM5
Connections:
- new net: U?.1 (VIN), U?.3 (EN)
- new net +5V: U?.5 (VOUT)
- new net GND: U?.2 (GND)
Changed lines of the file:
@@
 EESchema Schematic File Version 2
-LIBS:TLV2252AID
 LIBS:Power
 LIBS:Resistances_SMD_0603
@@
 LIBS:Microcontroleur_Atmel_SMD_TQFP
 LIBS:Barrettes_TH
+LIBS:Amplificateur_Operationel_SMD_SOIC
+LIBS:Quartz_SMD
+LIBS:Regulateurs_SMD_SOT89
+LIBS:Regulateurs_SMD_SOT23
 LIBS:LO2SC-cache
 EELAYER 25 0
@@
 	0    1    1    0
 $EndComp
+$Comp
+L MIC5205-3.3YM5 U?
+U 1 1 5601439B
+P 6150 3300
+F 0 "U?" H 5900 3500 50  0000 L CNN
+F 1 "MIC5205-3.3YM5" H 6150 3500 50  0000 L CNN
+F 2 "SOT23-5" H 6150 3300 50  0001 L CNN
+F 3 "" H 6150 3300 60  0000 C CNN
+	1    6150 3300
+	1    0    0    -1
+$EndComp
+$Comp
+L +5V #PWR?
+U 1 1 56014444
+P 6850 3100
+F 0 "#PWR?" H 6850 2950 50  0001 C CNN
+F 1 "+5V" H 6850 3240 50  0000 C CNN
+F 2 "" H 6850 3100 60  0000 C CNN
+F 3 "" H 6850 3100 60  0000 C CNN
+	1    6850 3100
+	1    0    0    -1
+$EndComp
+Wire Wire Line
+	6550 3200 6850 3200
+Wire Wire Line
+	6850 3200 6850 3100
+Wire Wire Line
+	5750 3300 5650 3300
+Wire Wire Line
+	5650 3300 5650 3200
+Wire Wire Line
+	5650 3200 5750 3200
+$Comp
+L GND #PWR?
+U 1 1 5601446C
+P 5650 3500
+F 0 "#PWR?" H 5650 3250 50  0001 C CNN
+F 1 "GND" H 5650 3350 50  0000 C CNN
+F 2 "" H 5650 3500 60  0000 C CNN
+F 3 "" H 5650 3500 60  0000 C CNN
+	1    5650 3500
+	1    0    0    -1
+$EndComp
+Wire Wire Line
+	5750 3400 5650 3400
+Wire Wire Line
+	5650 3400 5650 3500
 $EndSCHEMATC

Commit message: ??
Parts:
- removed U?: MIC5205-3.3YM5, SOT23-5, symbol MIC5205-3.3YM5
- added P3: CONN_01X10, Connecteurs_JAE:JAE_10Pins, symbol CONN_01X10
Changed lines of the file:
@@
 LIBS:Regulateurs_SMD_SOT89
 LIBS:Regulateurs_SMD_SOT23
+LIBS:Connecteurs_JAE_TH
 LIBS:LO2SC-cache
 EELAYER 25 0
@@
 $EndComp
 $Comp
-L MIC5205-3.3YM5 U?
-U 1 1 5601439B
-P 6150 3300
-F 0 "U?" H 5900 3500 50  0000 L CNN
-F 1 "MIC5205-3.3YM5" H 6150 3500 50  0000 L CNN
-F 2 "SOT23-5" H 6150 3300 50  0001 L CNN
-F 3 "" H 6150 3300 60  0000 C CNN
-	1    6150 3300
-	1    0    0    -1
+L CONN_01X10 P3
+U 1 1 56025E93
+P 6450 5200
+F 0 "P3" H 6450 5750 50  0000 C CNN
+F 1 "CONN_01X10" V 6550 5200 50  0000 C CNN
+F 2 "Connecteurs_JAE:JAE_10Pins" H 6450 5200 60  0001 C CNN
+F 3 "" H 6450 5200 60  0000 C CNN
+	1    6450 5200
+	0    -1   -1   0
 $EndComp
-$Comp
-L +5V #PWR?
-U 1 1 56014444
-P 6850 3100
-F 0 "#PWR?" H 6850 2950 50  0001 C CNN
-F 1 "+5V" H 6850 3240 50  0000 C CNN
-F 2 "" H 6850 3100 60  0000 C CNN
-F 3 "" H 6850 3100 60  0000 C CNN
-	1    6850 3100
-	1    0    0    -1
-$EndComp
-Wire Wire Line
-	6550 3200 6850 3200
-Wire Wire Line
-	6850 3200 6850 3100
-Wire Wire Line
-	5750 3300 5650 3300
-Wire Wire Line
-	5650 3300 5650 3200
-Wire Wire Line
-	5650 3200 5750 3200
-$Comp
-L GND #PWR?
-U 1 1 5601446C
-P 5650 3500
-F 0 "#PWR?" H 5650 3250 50  0001 C CNN
-F 1 "GND" H 5650 3350 50  0000 C CNN
-F 2 "" H 5650 3500 60  0000 C CNN
-F 3 "" H 5650 3500 60  0000 C CNN
-	1    5650 3500
-	1    0    0    -1
-$EndComp
-Wire Wire Line
-	5750 3400 5650 3400
-Wire Wire Line
-	5650 3400 5650 3500
 $EndSCHEMATC

Commit message: ?
Connections:
- net +5V: now reaches P1.5 (P5)
Changed lines of the file:
@@
 	0    -1   -1   0
 $EndComp
+$Comp
+L +5V #PWR?
+U 1 1 56030C63
+P 5950 1800
+F 0 "#PWR?" H 5950 1650 50  0001 C CNN
+F 1 "+5V" H 5950 1940 50  0000 C CNN
+F 2 "" H 5950 1800 60  0000 C CNN
+F 3 "" H 5950 1800 60  0000 C CNN
+	1    5950 1800
+	1    0    0    -1
+$EndComp
 $EndSCHEMATC

Commit message: ?
Connections:
- net labels added: +9V, 2.5v, CSEL0, CSEL1, CSEL2, DSEL, GND, H+, H-, IP, LATCH, PIN_VS, RCAL, SCLK, SIN
- wire segments 0 -> 11
Changed lines of the file:
@@
 $EndComp
 $Comp
-L +5V #PWR?
+L +5V #PWR01
 U 1 1 56030C63
 P 5950 1800
-F 0 "#PWR?" H 5950 1650 50  0001 C CNN
+F 0 "#PWR01" H 5950 1650 50  0001 C CNN
 F 1 "+5V" H 5950 1940 50  0000 C CNN
 F 2 "" H 5950 1800 60  0000 C CNN
@@
 	1    0    0    -1
 $EndComp
+Wire Wire Line
+	6050 1800 6050 1700
+Text GLabel 6050 1700 1    50   Input ~ 0
+DSEL
+Wire Wire Line
+	6150 1800 6150 1700
+Wire Wire Line
+	6250 1800 6250 1700
+Wire Wire Line
+	6350 1800 6350 1700
+Text GLabel 6150 1700 1    50   Input ~ 0
+CSEL2
+Text GLabel 6250 1700 1    50   Input ~ 0
+SCLK
+Text GLabel 6350 1700 1    50   Input ~ 0
+SIN
+$Comp
+L GND #PWR02
+U 1 1 5603DF84
+P 6800 1750
+F 0 "#PWR02" H 6800 1500 50  0001 C CNN
+F 1 "GND" H 6800 1600 50  0000 C CNN
+F 2 "" H 6800 1750 60  0000 C CNN
+F 3 "" H 6800 1750 60  0000 C CNN
+	1    6800 1750
+	-1   0    0    1
+$EndComp
+Wire Wire Line
+	6900 1750 6900 1650
+Wire Wire Line
+	7000 1750 7000 1650
+Wire Wire Line
+	7100 1750 7100 1650
+Wire Wire Line
+	7200 1750 7200 1650
+Text GLabel 7100 1650 1    50   Input ~ 0
+CSEL0
+Text GLabel 7000 1650 1    50   Input ~ 0
+CSEL1
+Text GLabel 7200 1650 1    50   Input ~ 0
+LATCH
+Wire Wire Line
+	6200 5400 6200 5900
+$Comp
+L +9V #PWR03
+U 1 1 5603EA59
+P 6200 5900
+F 0 "#PWR03" H 6200 5750 50  0001 C CNN
+F 1 "+9V" H 6200 6040 50  0000 C CNN
+F 2 "" H 6200 5900 60  0000 C CNN
+F 3 "" H 6200 5900 60  0000 C CNN
+	1    6200 5900
+	-1   0    0    1
+$EndComp
+Text GLabel 6300 5400 3    50   Input ~ 0
+PIN_VS
+Text GLabel 6000 5400 3    50   Input ~ 0
+2.5v
+Text GLabel 6100 5400 3    50   Input ~ 0
+IP
+Text GLabel 6700 5400 3    50   Input ~ 0
+RCAL
+Text GLabel 6600 5800 3    50   Input ~ 0
+H+
+Text GLabel 6900 5400 3    50   Input ~ 0
+H-
+$Comp
+L GND #PWR04
+U 1 1 5603F1CE
+P 6800 5400
+F 0 "#PWR04" H 6800 5150 50  0001 C CNN
+F 1 "GND" H 6800 5250 50  0000 C CNN
+F 2 "" H 6800 5400 60  0000 C CNN
+F 3 "" H 6800 5400 60  0000 C CNN
+	1    6800 5400
+	1    0    0    -1
+$EndComp
+Wire Wire Line
+	6600 5400 6600 5800
+Wire Wire Line
+	6200 5750 6600 5750
+Connection ~ 6600 5750
+Connection ~ 6200 5750
 $EndSCHEMATC
