File: PCB/Out_Lineat+WideBand.sch (KiCad schematic (older format))
At the start: 6 parts

Commit message: - ajout de schematiques
Parts:
- U1: renamed from U?; footprint SOIC127P600X175-8N -> Amplificateur_Operationel:SOIC127P600X175-8N
Connections:
- net OUT1 renamed 2.5v
Changed lines of the file:
@@
 LIBS:Resistances_SMD_0603
 LIBS:Condensateurs_SMD_0603
+LIBS:Microcontroleur_Atmel_SMD_TQFP
+LIBS:Barrettes_TH
 LIBS:LO2SC-cache
 EELAYER 25 0
@@
 $Descr A4 11693 8268
 encoding utf-8
-Sheet 2 2
+Sheet 2 5
 Title ""
 Date ""
@@
 	4050 3050 3650 3050
 Text GLabel 6000 3250 2    50   Input ~ 0
-OUT1
+2.5v
 Text GLabel 4050 2750 0    50   Input ~ 0
-OUT1
+2.5v
 $Comp
 L 1.2k R3
@@
 	2300 2950 2050 2950
 $Comp
-L TLV2252AID U?
+L TLV2252AID U1
 U 1 1 55FBAF48
 P 4850 2750
-F 0 "U?" H 4639 3309 50  0000 L CNN
+F 0 "U1" H 4639 3309 50  0000 L CNN
 F 1 "TLV2252AID" H 4778 1835 50  0000 L CNN
-F 2 "SOIC127P600X175-8N" H 4850 2750 50  0001 L CNN
+F 2 "Amplificateur_Operationel:SOIC127P600X175-8N" H 4850 2750 50  0001 L CNN
 F 3 "" H 4850 2750 60  0000 C CNN
 	1    4850 2750
