File: PCB/LO2SC.kicad_pcb (KiCad board)
At the start: 2 copper layers, 6 parts, among them U1 TLV2252AID

Commit message: - ajout de schematiques
Parts:
- added C3: 10nF, condensateurs:C_0603_HandSoldering, F.Cu at (92.0, 120.6)
- added C4: 100nF, condensateurs:C_0603_HandSoldering, F.Cu at (92.0, 120.6)
- added P1: CONN_01X05, Barrettes:Pin_Header_Straight_1x05, F.Cu at (76.0, 141.0)
- added P2: CONN_01X05, Barrettes:Pin_Header_Straight_1x05, F.Cu at (76.0, 137.5)
- added R10, R11, R9: 10k, resistances:R_0603_HandSoldering, F.Cu at (92.0, 120.6)
- added R4: 470k, resistances:R_0603_HandSoldering, F.Cu at (92.0, 120.6)
- added R5: 22k, resistances:R_0603_HandSoldering, F.Cu at (92.0, 120.6)
- added R6: 330k, resistances:R_0603_HandSoldering, F.Cu at (92.0, 120.6)
- added R7: 62, resistances:R_0603_HandSoldering, F.Cu at (92.0, 120.6)
- added R8: 47k, resistances:R_0603_HandSoldering, F.Cu at (92.0, 120.6)
- added Ref**: Val**, PCB:vue3D, F.Cu at (81.0, 121.0)
- added U2: MCU-ATMEGA328P-AU(TQFP32), atmel:TQFP32-0.8-7X7MM, F.Cu at (92.0, 120.6)
- added U3: TLV2252AID, Amplificateur_Operationel:SOIC127P600X175-8N, F.Cu at (81.0, 111.5)
- moved R1 94.9 mm to (71.7, 115.1)
- moved C2 79.1 mm to (92.0, 120.6)
- moved R3 78.1 mm to (92.0, 120.6)
- moved R2 70.6 mm to (92.0, 120.6)
- moved C1 69.7 mm to (92.0, 120.6)
- moved U1 58.1 mm to (92.0, 120.6)
Connections:
- net OUT1 renamed 2.5v
Other:
- board outline added: 48 x 48 mm
- net class Default: clearance 0.2 -> 0.25
- rule trace_clearance: 0.2 -> 0.25
- rule trace_min: 0.2 -> 0.25

Commit message: -
Parts:
- removed Ref**: Val**, PCB:vue3D
- moved R5 30.7 mm to (61.5, 117.5)
- moved R6 30.0 mm to (62.0, 122.0)
- moved R10 29.1 mm to (66.5, 106.5)
- moved C2 28.8 mm to (64.0, 127.5)
- moved R11 28.5 mm to (64.5, 113.0)
- moved R9 27.0 mm to (71.5, 103.0)
- moved R4 24.9 mm to (69.5, 110.0)
- moved C4 22.8 mm to (71.0, 129.5)
- moved R8 22.1 mm to (78.0, 103.5)
- moved R2 21.5 mm to (70.5, 120.5)
- moved C1 21.3 mm to (71.0, 124.0)
- moved R7 16.7 mm to (87.5, 104.5)
- moved U1 15.0 mm to (80.0, 129.5)
- moved C3 11.1 mm to (92.0, 109.5)
- moved R3 6.58 mm to (95.5, 115.0)
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Connections:
- R1 pad 2: (no net) -> POUT_WIDE
- R10 pad 1: (no net) -> POUT_VS
- R4 pad 2: (no net) -> POUT_IP
- R8 pad 1: (no net) -> POUT_NARROW
- U2 pad 10: (no net) -> POUT_IP
- U2 pad 11: (no net) -> POUT_VS
- U2 pad 13: (no net) -> POUT_WIDE
- U2 pad 18: (no net) -> +5V
- U2 pad 21: (no net) -> GND
- U2 pad 3: (no net) -> GND
- U2 pad 32: (no net) -> POUT_NARROW
- U2 pad 4: (no net) -> +5V
- U2 pad 5: (no net) -> GND
- U2 pad 6: (no net) -> +5V
Changed lines of the file:
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@@
-(kicad_pcb (version 4) (host pcbnew "(2015-08-26 BZR 6129, Git 2e41367)-product")
+(kicad_pcb (version 4) (host pcbnew "(2015-09-03 BZR 6154, Git 4636d8d)-product")
   (general
-    (links 31)
-    (no_connects 23)
+    (links 41)
+    (no_connects 41)
     (area 56.924999 96.924999 105.075001 145.075001)
     (thickness 1.6)
@@
     (tracks 0)
     (zones 0)
-    (modules 21)
-    (nets 15)
+    (modules 20)
+    (nets 19)
   )
   (page A4)
@@
   (net 13 OUT_NARROWBAND)
   (net 14 OUT_LINEAR)
+  (net 15 POUT_WIDE)
+  (net 16 POUT_IP)
+  (net 17 POUT_NARROW)
+  (net 18 POUT_VS)
   (net_class Default "Ceci est la Netclass par défaut"
     (clearance 0.25)
@@
     (add_net PIN_IPA)
     (add_net PIN_VS)
+    (add_net POUT_IP)
+    (add_net POUT_NARROW)
+    (add_net POUT_VS)
+    (add_net POUT_WIDE)
     (add_net RCAL)
   )
@@
     (pad 1 smd rect (at -1.1 0) (size 1.2 0.9) (layers F.Cu F.Paste F.Mask)
       (net 3 "Net-(C1-Pad1)"))
-    (pad 2 smd rect (at 1.1 0) (size 1.2 0.9) (layers F.Cu F.Paste F.Mask))
+    (pad 2 smd rect (at 1.1 0) (size 1.2 0.9) (layers F.Cu F.Paste F.Mask)
+      (net 15 POUT_WIDE))
     (model resistances/resistances.pretty/3dpackage/R_0603_HandSoldering.wrl
       (at (xyz 0 0 0))
@@
   )
   (module condensateurs:C_0603_HandSoldering (layer F.Cu)
-    (at 92 120.575001)
+    (at 71 124)
     (descr "Capacitor SMD 0603, hand soldering")
     (tags "capacitor 0603")
@@
   )
   (module condensateurs:C_0603_HandSoldering (layer F.Cu)
-    (at 92 120.575001)
+    (at 64 127.5)
     (descr "Capacitor SMD 0603, hand soldering")
     (tags "capacitor 0603")
@@
   )
   (module condensateurs:C_0603_HandSoldering (layer F.Cu)
-    (at 92 120.575001)
+    (at 92 109.5)
     (descr "Capacitor SMD 0603, hand soldering")
     (tags "capacitor 0603")
@@
   )
   (module condensateurs:C_0603_HandSoldering (layer F.Cu)
-    (at 92 120.575001)
+    (at 71 129.5)
     (descr "Capacitor SMD 0603, hand soldering")
     (tags "capacitor 0603")
@@
   )
   (module resistances:R_0603_HandSoldering (layer F.Cu)
-    (at 92 120.575001)
+    (at 70.5 120.5)
     (descr "Resistor SMD 0603, hand soldering")
     (tags "resistor 0603")
@@
   )
   (module resistances:R_0603_HandSoldering (layer F.Cu)
-    (at 92 120.575001)
+    (at 95.5 115)
     (descr "Resistor SMD 0603, hand soldering")
     (tags "resistor 0603")
@@
   )
   (module resistances:R_0603_HandSoldering (layer F.Cu)
-    (at 92 120.575001)
+    (at 69.5 110)
     (descr "Resistor SMD 0603, hand soldering")
     (tags "resistor 0603")
@@
     (pad 1 smd rect (at -1.1 0) (size 1.2 0.9) (layers F.Cu F.Paste F.Mask)
       (net 5 "Net-(C3-Pad1)"))
-    (pad 2 smd rect (at 1.1 0) (size 1.2 0.9) (layers F.Cu F.Paste F.Mask))
-    (model resistances/resistances.pretty/3dpackage/R_0603_HandSoldering.wrl
-      (at (xyz 0 0 0))
-      (scale (xyz 1 1 1))
-      (rotate (xyz 0 0 0))
-    )
-  )
-  (module resistances:R_0603_HandSoldering (layer F.Cu)
-    (at 92 120.575001)
+    (pad 2 smd rect (at 1.1 0) (size 1.2 0.9) (layers F.Cu F.Paste F.Mask)
+      (net 16 POUT_IP))
+    (model resistances/resistances.pretty/3dpackage/R_0603_HandSoldering.wrl
+      (at (xyz 0 0 0))
+      (scale (xyz 1 1 1))
+      (rotate (xyz 0 0 0))
+    )
+  )
+  (module resistances:R_0603_HandSoldering (layer F.Cu)
+    (at 61.5 117.5)
     (descr "Resistor SMD 0603, hand soldering")
     (tags "resistor 0603")
@@
   )
   (module resistances:R_0603_HandSoldering (layer F.Cu)
-    (at 92 120.575001)
+    (at 62 122)
     (descr "Resistor SMD 0603, hand soldering")
     (tags "resistor 0603")
@@
   )
   (module resistances:R_0603_HandSoldering (layer F.Cu)
-    (at 92 120.575001)
+    (at 87.5 104.5)
     (descr "Resistor SMD 0603, hand soldering")
     (tags "resistor 0603")
@@
   )
   (module resistances:R_0603_HandSoldering (layer F.Cu)
-    (at 92 120.575001)
+    (at 78 103.5)
     (descr "Resistor SMD 0603, hand soldering")
     (tags "resistor 0603")
@@
     (fp_line (start 0.5 0.675) (end -0.5 0.675) (layer F.SilkS) (width 0.15))
     (fp_line (start -0.5 -0.675) (end 0.5 -0.675) (layer F.SilkS) (width 0.15))
-    (pad 1 smd rect (at -1.1 0) (size 1.2 0.9) (layers F.Cu F.Paste F.Mask))
+    (pad 1 smd rect (at -1.1 0) (size 1.2 0.9) (layers F.Cu F.Paste F.Mask)
+      (net 17 POUT_NARROW))
     (pad 2 smd rect (at 1.1 0) (size 1.2 0.9) (layers F.Cu F.Paste F.Mask)
       (net 13 OUT_NARROWBAND))
@@
   )
   (module resistances:R_0603_HandSoldering (layer F.Cu)
-    (at 92 120.575001)
+    (at 71.5 103)
     (descr "Resistor SMD 0603, hand soldering")
     (tags "resistor 0603")
@@
   )
   (module resistances:R_0603_HandSoldering (layer F.Cu)
-    (at 92 120.575001)
+    (at 66.5 106.5)
     (descr "Resistor SMD 0603, hand soldering")
     (tags "resistor 0603")
@@
     (fp_line (start 0.5 0.675) (end -0.5 0.675) (layer F.SilkS) (width 0.15))
     (fp_line (start -0.5 -0.675) (end 0.5 -0.675) (layer F.SilkS) (width 0.15))
-    (pad 1 smd rect (at -1.1 0) (size 1.2 0.9) (layers F.Cu F.Paste F.Mask))
+    (pad 1 smd rect (at -1.1 0) (size 1.2 0.9) (layers F.Cu F.Paste F.Mask)
+      (net 18 POUT_VS))
     (pad 2 smd rect (at 1.1 0) (size 1.2 0.9) (layers F.Cu F.Paste F.Mask)
       (net 7 "Net-(C4-Pad2)"))
@@
   )
   (module resistances:R_0603_HandSoldering (layer F.Cu)
-    (at 92 120.575001)
+    (at 64.5 113)
     (descr "Resistor SMD 0603, hand soldering")
     (tags "resistor 0603")
@@
   )
   (module Amplificateur_Operationel:SOIC127P600X175-8N (layer F.Cu)
-    (at 92 120.575001)
+    (at 80 129.5)
     (solder_mask_margin 0.1)
     (attr smd)
@@
   )
   (module atmel:TQFP32-0.8-7X7MM (layer F.Cu)
-    (at 92 120.575001)
+    (at 91 123.5)
     (descr "<B>Thin Plasic Quad Flat Package</B> Grid 0.8 mm")
     (solder_mask_margin 0.1)
@@
       (solder_mask_margin 0.2))
     (pad 3 smd rect (at -4.2926 -1.2) (size 1.27 0.5588) (layers F.Cu F.Paste F.Mask)
-      (solder_mask_margin 0.2))
+      (net 1 GND) (solder_mask_margin 0.2))
     (pad 4 smd rect (at -4.2926 -0.4) (size 1.27 0.5588) (layers F.Cu F.Paste F.Mask)
-      (solder_mask_margin 0.2))
+      (net 2 +5V) (solder_mask_margin 0.2))
     (pad 5 smd rect (at -4.2926 0.4) (size 1.27 0.5588) (layers F.Cu F.Paste F.Mask)
-      (solder_mask_margin 0.2))
+      (net 1 GND) (solder_mask_margin 0.2))
     (pad 6 smd rect (at -4.2926 1.2) (size 1.27 0.5588) (layers F.Cu F.Paste F.Mask)
-      (solder_mask_margin 0.2))
+      (net 2 +5V) (solder_mask_margin 0.2))
     (pad 7 smd rect (at -4.2926 2) (size 1.27 0.5588) (layers F.Cu F.Paste F.Mask)
       (solder_mask_margin 0.2))
@@
       (solder_mask_margin 0.2))
     (pad 10 smd rect (at -2 4.2926) (size 0.5588 1.27) (layers F.Cu F.Paste F.Mask)
-      (solder_mask_margin 0.2))
+      (net 16 POUT_IP) (solder_mask_margin 0.2))
     (pad 11 smd rect (at -1.2 4.2926) (size 0.5588 1.27) (layers F.Cu F.Paste F.Mask)
-      (solder_mask_margin 0.2))
+      (net 18 POUT_VS) (solder_mask_margin 0.2))
     (pad 12 smd rect (at -0.4 4.2926) (size 0.5588 1.27) (layers F.Cu F.Paste F.Mask)
       (solder_mask_margin 0.2))
     (pad 13 smd rect (at 0.4 4.2926) (size 0.5588 1.27) (layers F.Cu F.Paste F.Mask)
-      (solder_mask_margin 0.2))
+      (net 15 POUT_WIDE) (solder_mask_margin 0.2))
     (pad 14 smd rect (at 1.2 4.2926) (size 0.5588 1.27) (layers F.Cu F.Paste F.Mask)
       (solder_mask_margin 0.2))
@@
       (solder_mask_margin 0.2))
     (pad 18 smd rect (at 4.2926 2) (size 1.27 0.5588) (layers F.Cu F.Paste F.Mask)
-      (solder_mask_margin 0.2))
+      (net 2 +5V) (solder_mask_margin 0.2))
     (pad 19 smd rect (at 4.2926 1.2) (size 1.27 0.5588) (layers F.Cu F.Paste F.Mask)
       (solder_mask_margin 0.2))
@@
       (solder_mask_margin 0.2))
     (pad 21 smd rect (at 4.2926 -0.4) (size 1.27 0.5588) (layers F.Cu F.Paste F.Mask)
-      (solder_mask_margin 0.2))
+      (net 1 GND) (solder_mask_margin 0.2))
     (pad 22 smd rect (at 4.2926 -1.2) (size 1.27 0.5588) (layers F.Cu F.Paste F.Mask)
       (solder_mask_margin 0.2))
@@
       (solder_mask_margin 0.2))
     (pad 32 smd rect (at -2.8 -4.2926) (size 0.5588 1.27) (layers F.Cu F.Paste F.Mask)
-      (solder_mask_margin 0.2))
+      (net 17 POUT_NARROW) (solder_mask_margin 0.2))
     (model "Circuit Intégré/Microcontroleur/Atmel/atmel.pretty/3dPackage/TQFP-32_7x7mm_Pitch0-8mm.wrl"
       (at (xyz 0 0 0))
@@
       (rotate (xyz 0 0 0))
     )
-  )
-  (module PCB:vue3D (layer F.Cu)
-    (at 81 121)
-    (attr smd)
-    (fp_text reference Ref** (at 4.5 -24.5) (layer F.SilkS) hide
-      (effects (font (size 1 1) (thickness 0.15)))
-    )
-    (fp_text value Val** (at -0.5 -24.5) (layer F.Fab) hide
-      (effects (font (size 1 1) (thickness 0.15)))
-    )
-    (fp_circle (center 0 0) (end -24 0) (layer F.SilkS) (width 0.15))
-    (model C:/Users/ARRT/Documents/Github/Universal_Display_Automotive/PCB/UDA.wrl
-      (at (xyz 0 0 -0.35))
-      (scale (xyz 0.39 0.39 0.39))
-      (rotate (xyz 0 0 0))
-    )

Commit message: - premier test avec l'arduino
Parts:
- added Ref**: Val**, PCB:vue3D, F.Cu at (81.0, 121.0)
- moved R11 33.6 mm to (94.0, 129.0), turned to 270 degrees
- moved R6 29.2 mm to (87.0, 107.0), turned to 270 degrees
- moved R5 24.8 mm to (83.5, 106.0), turned to 180 degrees
- moved C4 23.6 mm to (94.0, 124.0), turned to 270 degrees
- moved U1 22.1 mm to (100.0, 120.0)
- moved C3 12.7 mm to (80.5, 115.0), turned to 90 degrees
- moved U2 8.25 mm to (83.0, 125.5)
- moved R7 5.32 mm to (83.5, 108.0)
- moved U3 5.32 mm to (85.0, 115.0)

Commit message: - routage
Parts:
- removed Ref**: Val**, PCB:vue3D
- added C5: 100nF, condensateurs:C_0603_HandSoldering, F.Cu at (77.5, 122.5)
- added C6: 1nF, condensateurs:C_0603_HandSoldering, F.Cu at (64.0, 130.5)
- added C7: 1nF, condensateurs:C_0603_HandSoldering, F.Cu at (62.5, 111.0)
- added C8: 100nF, condensateurs:C_0603_HandSoldering, F.Cu at (74.0, 112.5)
- added R12: 10k, resistances:R_0603_HandSoldering, F.Cu at (72.0, 112.5)
- added U4: ABLS2-16.000MHZ-D4Y-T, Quartz:HC-49, F.Cu at (61.0, 121.5)
- moved R1 28.6 mm to (98.5, 125.0)
- moved C1 27.7 mm to (98.5, 127.0)
- moved R11 25.9 mm to (68.5, 133.5), turned to 180 degrees
- moved R10 24.1 mm to (68.5, 130.5)
- moved C4 21.0 mm to (74.0, 130.5), turned to 180 degrees
- moved R4 19.9 mm to (89.0, 106.0)
- moved R3 18.4 mm to (82.5, 128.0), turned to 90 degrees
- moved C2 17.2 mm to (79.0, 119.0), turned to 90 degrees
- moved U2 14.4 mm to (69.0, 122.0)
- moved R6 13.9 mm to (73.5, 103.5), turned to 90 degrees
- moved R8 13.8 mm to (68.0, 113.0)
- moved R5 13.6 mm to (70.0, 104.5)
- moved R2 12.4 mm to (82.5, 123.5), turned to 90 degrees
- moved U3 11.2 mm to (81.0, 104.5), turned to 0 degrees
- moved C3 11.0 mm to (89.0, 108.0), turned to 0 degrees
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Connections:
- U2 pad 20: (no net) -> Net-(C5-Pad1)
- U2 pad 29: (no net) -> Net-(C8-Pad1)
- U2 pad 7: (no net) -> Net-(C7-Pad2)
- U2 pad 8: (no net) -> Net-(C6-Pad2)
Routing:
- net +5V: track 0.00 -> 104.6 mm, vias 0 -> 2
- net POUT_IP: track 0.00 -> 67.7 mm, vias 0 -> 2
- net POUT_WIDE: track 0.00 -> 42.4 mm, vias 0 -> 2
- net IP: track 0.00 -> 36.1 mm, vias 0 -> 2
- net PIN_IPA: track 0.00 -> 26.6 mm, vias 0 -> 2
- net 2.5v: track 0.00 -> 17.2 mm
- net PIN_VS: track 0.00 -> 15.4 mm, vias 0 -> 2
- net Net-(C7-Pad2): track 0.00 -> 14.9 mm
- net RCAL: track 0.00 -> 13.0 mm
- net Net-(C6-Pad2): track 0.00 -> 10.3 mm
- net Net-(R2-Pad1): track 0.00 -> 8.53 mm
- net Net-(C8-Pad1): track 0.00 -> 8.52 mm
- net Net-(R5-Pad1): track 0.00 -> 7.78 mm
- net Net-(C3-Pad1): track 0.00 -> 6.67 mm
- net Net-(C4-Pad2): track 0.00 -> 6.45 mm
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- added copper zone on F.Cu, net GND

Commit message: ??
Parts:
- added P3: CONN_01X10, Connecteurs_JAE:JAE_10Pins, F.Cu at (103.5, 98.0)
Changed lines of the file:
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@@
     (links 53)
     (no_connects 0)
-    (area 101.174999 92.674999 149.325001 140.825001)
+    (area 56.924999 96.924999 105.075001 145.075001)
     (thickness 1.6)
     (drawings 2)
     (tracks 138)
     (zones 0)
-    (modules 26)
+    (modules 27)
     (nets 23)
   )
@@
   )
   (setup
-    (last_trace_width 0.5)
+    (last_trace_width 0.25)
     (user_trace_width 0.3)
     (user_trace_width 0.4)
@@
     )
   )
+  (module Connecteurs_JAE:JAE_10Pins (layer F.Cu)
+    (at 103.5 98)
+    (descr "Through hole pin header")
+    (tags "pin header")
+    (fp_text reference P3 (at 0.21 -8.97) (layer F.SilkS)
+      (effects (font (size 1 1) (thickness 0.15)))
+    )
+    (fp_text value CONN_01X10 (at 0.11 -10.66) (layer F.SilkS)
+      (effects (font (size 1 1) (thickness 0.15)))
+    )
+    (fp_circle (center 0.02 0.035) (end -7.63 0.985) (layer F.SilkS) (width 0.2))
+    (pad 1 thru_hole circle (at -2.37886 -2.11908) (size 2.1844 2.1844) (drill 1.39954) (layers *.Cu *.Mask F.SilkS))
+    (pad 2 thru_hole circle (at 3.61808 0.02976) (size 2.1844 2.1844) (drill 1.39954) (layers *.Cu *.Mask F.SilkS))
+    (pad 3 thru_hole circle (at 2.4192 -2.11908) (size 2.1844 2.1844) (drill 1.39954) (layers *.Cu *.Mask F.SilkS))
+    (pad 4 thru_hole circle (at 0.0189 -2.11908) (size 2.1844 2.1844) (drill 1.39954) (layers *.Cu *.Mask F.SilkS))
+    (pad 5 thru_hole circle (at -3.58028 0.02976) (size 2.1844 2.1844) (drill 1.39954) (layers *.Cu *.Mask F.SilkS))
+    (pad 6 thru_hole circle (at 2.4192 2.18114) (size 2.1844 2.1844) (drill 1.39954) (layers *.Cu *.Mask F.SilkS))
+    (pad 7 thru_hole circle (at 0.0189 2.18114) (size 2.1844 2.1844) (drill 1.39954) (layers *.Cu *.Mask F.SilkS))
+    (pad 8 thru_hole circle (at -2.37886 2.18114) (size 2.1844 2.1844) (drill 1.39954) (layers *.Cu *.Mask F.SilkS))
+    (pad 9 thru_hole circle (at 1.21778 0.02976) (size 2.1844 2.1844) (drill 1.39954) (layers *.Cu *.Mask F.SilkS))
+    (pad 10 thru_hole circle (at -1.17998 0.02976) (size 2.1844 2.1844) (drill 1.39954) (layers *.Cu *.Mask F.SilkS))
+  )
   (gr_circle (center 81 121) (end 57 121) (layer Edge.Cuts) (width 0.15))

Commit message: ?
Parts:
- added Ref**: Val**, PCB:vue3D, B.Cu at (81.0, 121.0)
- P3: moved to B.Cu
- moved P3 31.8 mm to (81.0, 120.5), turned to 180 degrees
- moved C7 25.5 mm to (80.5, 129.0), turned to 0 degrees
- moved C4 24.8 mm to (97.5, 122.5), turned to 90 degrees
- moved U2 24.5 mm to (92.5, 129.0)
- moved C5 24.4 mm to (101.0, 129.0)
- moved R10 23.6 mm to (90.5, 139.0)
- moved R11 23.2 mm to (90.5, 141.0)
- moved R8 22.8 mm to (89.5, 120.5), turned to 90 degrees
- moved R9 22.3 mm to (89.5, 116.0), turned to 90 degrees
- moved R3 21.6 mm to (84.5, 106.5), turned to 0 degrees
- moved R12 21.6 mm to (93.0, 117.5), turned to 180 degrees
- moved C2 20.8 mm to (91.0, 102.0), turned to 0 degrees
- moved U4 20.5 mm to (78.0, 133.0), turned to 0 degrees
- moved C8 19.2 mm to (93.0, 115.5), turned to 0 degrees
- moved R1 19.1 mm to (96.5, 106.0), turned to 90 degrees
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Connections:
- P1 pad 5: (no net) -> +5V
Routing:
- net IP: track 36.1 -> 7.34 mm, vias 2 -> 0
- net 2.5v: track 17.2 -> 42.3 mm, vias 0 -> 2
- net Net-(C4-Pad2): track 6.45 -> 29.1 mm, vias 0 -> 2
- net PIN_IPA: track 26.6 -> 49.2 mm
- net Net-(C6-Pad2): track 10.3 -> 31.5 mm
- net POUT_IP: track 67.7 -> 48.8 mm
- net PIN_VS: track 15.4 -> 3.34 mm, vias 2 -> 0
- net POUT_WIDE: track 42.4 -> 36.2 mm
- net Net-(C7-Pad2): track 14.9 -> 10.8 mm
- net Net-(R2-Pad1): track 8.53 -> 4.99 mm
- net OUT_NARROWBAND: track 3.00 -> 0.00 mm
- net POUT_VS: track 4.37 -> 6.49 mm
- net +5V: track 104.6 -> 106.7 mm, vias 2 -> 5
- net RCAL: track 13.0 -> 11.0 mm
- net POUT_NARROW: track 5.00 -> 3.19 mm
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
Commit message: ?
Parts:
- moved R9 4.25 mm to (87.5, 119.8)
- moved R8 3.72 mm to (87.0, 123.2), turned to 180 degrees
- moved C8 3.25 mm to (93.0, 112.2)
- moved R12 3.25 mm to (93.0, 114.2)
- moved C4 0.75 mm to (98.2, 122.5)
- moved R4 0.75 mm to (78.5, 108.2)
Connections:
- P1 pad 1: (no net) -> SIN
- P1 pad 2: (no net) -> SCLK
- P1 pad 3: (no net) -> CSEL2
- P1 pad 4: (no net) -> DSEL
- P2 pad 1: (no net) -> LATCH
- P2 pad 2: (no net) -> CSEL0
- P2 pad 3: (no net) -> CSEL1
- P2 pad 5: (no net) -> GND
- P3 pad 1: (no net) -> 2.5v
- P3 pad 2: (no net) -> IP
- P3 pad 3: (no net) -> H+
- P3 pad 4: (no net) -> PIN_VS
- P3 pad 7: (no net) -> H+
- P3 pad 8: (no net) -> RCAL
- P3 pad 9: (no net) -> GND
- U2 pad 1: (no net) -> SCLK
- U2 pad 15: (no net) -> DSEL
- U2 pad 16: (no net) -> CSEL2
- U2 pad 2: (no net) -> SIN
- U2 pad 26: (no net) -> CSEL1
- U2 pad 27: (no net) -> CSEL0
- U2 pad 28: (no net) -> LATCH
Routing:
- net RCAL: track 11.0 -> 64.8 mm, vias 0 -> 2
- net SCLK: track 0.00 -> 45.4 mm, vias 0 -> 1
- net LATCH: track 0.00 -> 41.0 mm, vias 0 -> 1
- net CSEL0: track 0.00 -> 36.6 mm, vias 0 -> 1
- net SIN: track 0.00 -> 35.9 mm, vias 0 -> 1
- net CSEL1: track 0.00 -> 31.3 mm, vias 0 -> 1
- net CSEL2: track 0.00 -> 25.4 mm, vias 0 -> 1
- net IP: track 7.34 -> 23.5 mm
- net DSEL: track 0.00 -> 16.2 mm, vias 0 -> 1
- net 2.5v: track 42.3 -> 58.4 mm, vias 2 -> 3
- net GND: track 0.00 -> 3.58 mm, vias 0 -> 1
- net Net-(C8-Pad1): track 9.35 -> 12.6 mm
- net +5V: track 106.7 -> 109.8 mm
- net OUT_NARROWBAND: track 0.00 -> 3.12 mm
- net H+: track 0.00 -> 2.65 mm
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
Commit message: - routage en cours
Parts:
- moved C4 2.46 mm to (100.5, 123.5), turned to 0 degrees
- moved C5 1.00 mm to (100.0, 129.0)
Routing:
- net PIN_VS: track 4.60 -> 28.9 mm, vias 0 -> 2
- net GND: track 3.58 -> 18.4 mm, vias 1 -> 3
- net LATCH: track 41.0 -> 32.8 mm
- net CSEL1: track 31.3 -> 25.5 mm
- net Net-(C4-Pad2): track 30.2 -> 25.4 mm, vias 2 -> 0
- net CSEL0: track 36.6 -> 31.9 mm
- net Net-(C5-Pad1): track 3.42 -> 2.42 mm
- net PIN_IPA: track 50.9 -> 51.4 mm
